File: hw/KiCAD/FD_PCB_Separate_Barrel/FD_PCB.kicad_pcb (KiCad board)
At the start: 2 copper layers, 231.2 x 136.6 mm, 144 parts, among them J1 Barrel_Jack_Switch, J10 Conn_01x02, J11 Conn_01x02, J12 Conn_01x02, J13 Conn_02x10_Odd_Even, J14 MQ-4 Gas Sensor, J15 MQ-7 Gas Sensor, J16 MQ-138 Gas Sensor, J17 KY-026 Flame Sensor, J18 Conn_01x10, J19 Conn_01x05, J2 Conn_02x12_Odd_Even, J20 HDC3022, J21 Conn_01x08, J22 MiCS-6814, J23 Conn_01x02, J3 Conn_02x12_Odd_Even, J4 Conn_02x20_Odd_Even, J5 Conn_02x10_Odd_Even, J6 Conn_01x07, J7 Conn_01x02, J8 Conn_01x08, J9 Conn_01x16, M1 Motor_Servo, M2 Motor_Servo, SW1 SW_Push, SW2 SW_Push, SW3 SW_Push, U1 ADS1115IDGS, U2 OPA2350, U3 OPA2350, U4 ADS1115IDGS

Commit message: finish adding mouting holes and do some prints
Parts:
- added H1: ~, ECE445L:MountingHole_4_40, F.Cu at (80.8, 109.6)
- added H2: ~, ECE445L:MountingHole_4_40, F.Cu at (80.8, 115.8)
- added H3: ~, ECE445L:MountingHole_4_40, F.Cu at (80.8, 121.9)
- added H4: ~, ECE445L:MountingHole_4_40, F.Cu at (80.8, 128.0)
- added J24: Conn_01x02, Connector_PinHeader_2.54mm:PinHeader_1x02_P2.54mm_Vertical, F.Cu at (37.0, 44.0)
- added J25: Conn_01x02, Connector_PinHeader_2.54mm:PinHeader_1x02_P2.54mm_Vertical, F.Cu at (20.9, 84.0)
- moved D1 94.5 mm to (169.0, 100.4)
- moved D2 94.5 mm to (169.0, 107.9)
- moved D3 94.5 mm to (169.0, 115.4)
- moved D4 94.5 mm to (169.0, 122.9)
- moved J21 94.5 mm to (176.2, 101.5)
- moved TP10 86.9 mm to (261.7, 116.8)
- moved TP12 86.9 mm to (261.7, 130.5)
- moved TP13 86.9 mm to (261.7, 135.1)
- moved TP14 86.9 mm to (261.7, 125.9)
- moved TP2 86.9 mm to (261.7, 112.2)
- moved TP3 86.9 mm to (261.7, 98.5)
- moved TP46 86.9 mm to (261.7, 93.9)
- moved TP5 86.9 mm to (261.7, 107.6)
- moved TP6 86.9 mm to (261.7, 103.1)
- moved TP7 86.9 mm to (261.7, 121.3)
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Connections:
- J1 pad 1: +5V_EXT -> Net-(J24-Pin_1)
- J1 pad 2: EXT_GND -> B_Jack_GND
Routing:
- net B_Jack_GND: track 0.00 -> 11.8 mm
- net EXT_GND: track 260.0 -> 251.7 mm
- net Net-(J24-Pin_1): track 0.00 -> 4.20 mm
- net +5V_EXT: track 162.0 -> 166.1 mm
Other:
- board size 231.2 x 136.6 mm -> 246.2 x 120.3 mm
- board text added: "V+"
- board text added: "V-"
- board text removed: "EXT_+5V"
