File: hw/KiCAD/FD_PCB_SB_No_Peninsula/FD_PCB.kicad_pcb (KiCad board)
At the start: 2 copper layers, 231.2 x 136.6 mm, 144 parts, among them J1 Barrel_Jack_Switch, J10 Conn_01x02, J11 Conn_01x02, J12 Conn_01x02, J13 Conn_02x10_Odd_Even, J14 MQ-4 Gas Sensor, J15 MQ-7 Gas Sensor, J16 MQ-138 Gas Sensor, J17 KY-026 Flame Sensor, J18 Conn_01x10, J19 Conn_01x05, J2 Conn_02x12_Odd_Even, J20 HDC3022, J21 Conn_01x08, J22 MiCS-6814, J23 Conn_01x02, J3 Conn_02x12_Odd_Even, J4 Conn_02x20_Odd_Even, J5 Conn_02x10_Odd_Even, J6 Conn_01x07, J7 Conn_01x02, J8 Conn_01x08, J9 Conn_01x16, M1 Motor_Servo, M2 Motor_Servo, SW1 SW_Push, SW2 SW_Push, SW3 SW_Push, U1 ADS1115IDGS, U2 OPA2350, U3 OPA2350, U4 ADS1115IDGS

Commit message: finish adding mouting holes and do some prints
Parts:
- added H1: ~, ECE445L:MountingHole_4_40, F.Cu at (169.7, 136.8)
- added H10: ~, ECE445L:MountingHole_4_40, F.Cu at (92.7, 162.9)
- added H11: ~, ECE445L:MountingHole_4_40, F.Cu at (241.0, 42.7)
- added H12: ~, ECE445L:MountingHole_4_40, F.Cu at (204.8, 102.2)
- added H13: ~, ECE445L:MountingHole_4_40, F.Cu at (160.5, 106.2)
- added H14: ~, ECE445L:MountingHole_4_40, F.Cu at (266.3, 42.7)
- added H15: ~, ECE445L:MountingHole_4_40, F.Cu at (266.3, 106.2)
- added H16: ~, ECE445L:MountingHole_4_40, F.Cu at (176.5, 42.8)
- added H17: ~, ECE445L:MountingHole_4_40, F.Cu at (113.8, 26.2)
- added H18: ~, ECE445L:MountingHole_4_40, F.Cu at (124.8, 26.2)
- added H19: ~, ECE445L:MountingHole_4_40, F.Cu at (23.0, 60.0)
- added H2: ~, ECE445L:MountingHole_4_40, F.Cu at (206.0, 136.8)
- added H3: ~, ECE445L:MountingHole_4_40, F.Cu at (120.2, 141.3)
- added H4: ~, ECE445L:MountingHole_4_40, F.Cu at (135.2, 141.3)
- added H5: ~, ECE445L:MountingHole_4_40, F.Cu at (120.2, 125.1)
- added H6: ~, ECE445L:MountingHole_4_40, F.Cu at (135.2, 125.1)
- added H7: ~, ECE445L:MountingHole_4_40, F.Cu at (27.0, 109.9)
- added H8: ~, ECE445L:MountingHole_4_40, F.Cu at (27.0, 162.9)
- added H9: ~, ECE445L:MountingHole_4_40, F.Cu at (92.7, 109.9)
- added J24: Conn_01x02, Connector_PinHeader_2.54mm:PinHeader_1x02_P2.54mm_Vertical, F.Cu at (133.7, 134.5)
- added J25: Conn_01x02, Connector_PinHeader_2.54mm:PinHeader_1x02_P2.54mm_Vertical, F.Cu at (20.9, 84.0)
- moved J1 141.7 mm to (130.0, 133.2), turned to -90 degrees
- moved D1 130.2 mm to (197.7, 134.4), turned to 0 degrees
- moved J21 124.7 mm to (196.6, 141.6), turned to -90 degrees
- moved D2 120.8 mm to (190.2, 134.4), turned to 0 degrees
- moved D3 111.5 mm to (182.7, 134.4), turned to 0 degrees
- moved D4 102.4 mm to (175.2, 134.4), turned to 0 degrees
- moved J9 84.9 mm to (81.5, 117.3)
- moved R1 84.9 mm to (30.1, 155.9)
- moved R3 84.9 mm to (27.6, 155.9)
- moved R4 84.9 mm to (25.0, 155.9)
- moved SW1 84.9 mm to (25.3, 130.4)
- moved SW2 84.9 mm to (25.3, 141.1)
- moved SW3 84.9 mm to (25.3, 151.8)
- moved TP1 84.9 mm to (87.3, 122.5)
- moved TP10 84.9 mm to (93.1, 139.1)
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Connections:
- J1 pad 1: +5V_EXT -> Net-(J24-Pin_1)
- J1 pad 2: EXT_GND -> B_Jack_GND
Routing:
- net B_Jack_GND: track 0.00 -> 11.8 mm
- net EXT_GND: track 260.0 -> 251.7 mm
- net Net-(J24-Pin_1): track 0.00 -> 4.20 mm
- net +5V_EXT: track 162.0 -> 166.1 mm
- net GND: track 136.1 -> 135.5 mm
Other:
- board size 231.2 x 136.6 mm -> 251.3 x 143.9 mm
- board text added: "FD PCB Layouts V2 - Separated Barrel, with Peninsula"
- board text added: "Reference Measurements"
- board text added: "V+"
- board text added: "V-"
- board text removed: "EXT_+5V"

Commit message: add silkscreen, generate latest print p3-104
Parts:
- added G***: LOGO, Images:Asparagus-h-stretch, F.Cu at (125.0, 52.8)
- added G***: LOGO, Images:FireIcon, F.Cu at (166.4, 66.8)
- added G***: LOGO, Images:Asparagus-quarter-size, F.Cu at (188.5, 57.1)
- moved R5 1.11 mm to (241.8, 105.2), turned to 180 degrees
- renumbered TP11 to GND
Other:
- board text added: "1_CTS"
- board text added: "3.3V"
- board text added: "40"
- board text added: "5.0V"
- board text added: "CS0"
- board text added: "CS1"
- board text added: "FD Jetson Header Board"
- board text added: "FD LCD BOARD"
- board text added: "GPIO01"
- board text added: "GPIO07"
- board text added: "GPIO09"
- board text added: "GPIO11"
- board text added: "GPIO12"
- board text added: "GPIO13"
- board text added: "Gas Sensor Array"
- board text added: "I2C0"
- board text added: "I2C0_SDA"
- board text added: "I2C1_SCL"
- board text added: "I2C1_SDA"
- board text added: "I2S0"
- board text added: "I2S0_FS"
- board text added: "JETSON HEADER CONN"
- board text added: "MISO"
- board text added: "PITCH SERVO"
- board text added: "RX1"
- board text added: "SCK"
- board text added: "SCL"
- board text added: "SEN0219 CONN"
- board text added: "SPI0"
- board text added: "SPI0_MISO"
- board text added: "SPI0_MOSI"
- board text added: "SPI0_SCK"
- board text added: "SPI1"
- board text added: "SPI1_MOSI"
- board text added: "SPI1_SCK"
- board text added: "TX1"
- board text added: "UART1"
- board text added: "UART1_RTS"
- board text added: "YAW SERVO"
- board text added: "p1"
- board text added: "p2"
- board text added: "p39"
