File: hw/KiCAD/FD_PCB_SB_With_Peninsula/FD_PCB.kicad_pcb (KiCad board)
At the start: 2 copper layers, 251.3 x 143.9 mm, 168 parts, among them J1 Barrel_Jack_Switch, J10 Conn_01x02, J11 Conn_01x02, J12 Conn_01x02, J13 Conn_02x10_Odd_Even, J14 MQ-4 Gas Sensor, J15 MQ-7 Gas Sensor, J16 MQ-138 Gas Sensor, J17 KY-026 Flame Sensor, J18 Conn_01x10, J19 Conn_01x05, J2 Conn_02x12_Odd_Even, J20 HDC3022, J21 Conn_01x08, J22 MiCS-6814, J23 Conn_01x02, J24 Conn_01x02, J25 Conn_01x02, J3 Conn_02x12_Odd_Even, J4 Conn_02x20_Odd_Even, J5 Conn_02x10_Odd_Even, J6 Conn_01x07, J7 Conn_01x02, J8 Conn_01x08, J9 Conn_01x16, M1 Motor_Servo, M2 Motor_Servo, SW1 SW_Push, SW2 SW_Push, SW3 SW_Push, U1 ADS1115IDGS, U2 OPA2350, U3 OPA2350, U4 ADS1115IDGS

Commit message: fix header board collision dimensions, add additional mounting hole on header board
Parts:
- added H20: ~, ECE445L:MountingHole_4_40, F.Cu at (123.0, 98.3)
- moved C17 1.34 mm to (131.1, 92.8)
- moved C19 1.34 mm to (118.2, 85.8)
- moved C20 1.34 mm to (118.3, 97.0)
- moved C3 1.34 mm to (111.4, 93.3)
- moved J10 1.34 mm to (127.9, 96.8)
- moved M1 1.34 mm to (122.1, 89.1)
- moved M2 1.34 mm to (122.1, 93.8)
- moved C2 1.34 mm to (111.4, 89.8)
- moved C16 1.34 mm to (127.8, 93.4)
- moved J4 1.30 mm to (115.5, 80.6)
- moved G*** 0.73 mm to (125.3, 53.5)
- moved C1 0.14 mm to (40.3, 80.8)
- renumbered GND to TP11
Routing:
- net GPIO13: track 63.6 -> 61.2 mm
- net EXT_GND: track 251.7 -> 250.1 mm
- net GPIO07: track 54.7 -> 53.1 mm
- net GPIO12: track 58.0 -> 56.6 mm
- net +5V_EXT: track 166.1 -> 164.7 mm
- net +5V: track 49.3 -> 50.6 mm
- net I2S0_DOUT: track 112.4 -> 111.1 mm
- net GPIO11: track 37.2 -> 35.9 mm
- net I2C1_SDA: track 58.7 -> 60.0 mm
- net GPIO09: track 25.1 -> 26.4 mm
- net UART1_TXD: track 46.9 -> 48.2 mm
- net I2S0_SCK: track 75.3 -> 74.0 mm
- net I2C1_SCL: track 58.2 -> 59.5 mm
- net GPIO01: track 36.1 -> 34.8 mm
- net SPI0_CS0: track 34.5 -> 33.8 mm
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Other:
- outline, holes or cut-outs redrawn
- board text added: "RXD"
- board text added: "TXD"
- board text removed: "RX1"
- board text removed: "TX1"
