File: hw/KiCAD/FD_PCB_SB_With_Peninsula/FD_PCB.kicad_sch (KiCad schematic)
At the start: 166 parts, among them J1 Barrel_Jack_Switch, J10 Conn_01x02, J11 Conn_01x02, J12 Conn_01x02, J13 Conn_02x10_Odd_Even, J14 MQ-4 Gas Sensor, J15 MQ-7 Gas Sensor, J16 MQ-138 Gas Sensor, J17 KY-026 Flame Sensor, J18 Conn_01x10, J19 Conn_01x05, J2 Conn_02x12_Odd_Even, J20 HDC3022, J21 Conn_01x08, J22 MiCS-6814, J23 Conn_01x02, J24 Conn_01x02, J25 Conn_01x02, J3 Conn_02x12_Odd_Even, J4 Conn_02x20_Odd_Even, J5 Conn_02x10_Odd_Even, J6 Conn_01x07, J7 Conn_01x02, J8 Conn_01x08, J9 Conn_01x16, M1 Motor_Servo, M2 Motor_Servo, SW1 SW_Push, SW2 SW_Push, SW3 SW_Push, U1 ADS1115IDGS, U2 OPA2350, U3 OPA2350, U4 ADS1115IDGS

Commit message: separate boards and generate pcb production gerber files
Connections:
- no-connect marks 33 -> 53
Changed lines of the file:
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@@
+	)
+	(no_connect
+		(at 346.71 19.05)
+	)
+	(no_connect
+		(at -1.27 121.92)
+	)
+	(no_connect
+		(at 5.08 43.18)
+	)
+	(no_connect
+		(at -1.27 115.57)
 	)
 	(no_connect
@@
 	)
 	(no_connect
+		(at 5.08 30.48)
+	)
+	(no_connect
 		(at 95.25 170.18)
+	)
+	(no_connect
+		(at 8.89 115.57)
 	)
 	(no_connect
@@
 	(no_connect
 		(at 95.25 167.64)
+	)
+	(no_connect
+		(at 374.65 162.56)
+	)
+	(no_connect
+		(at 354.33 162.56)
 	)
 	(no_connect
@@
 	)
 	(no_connect
+		(at 346.71 25.4)
+	)
+	(no_connect
 		(at -11.43 132.08)
 	)
@@
 	)
 	(no_connect
+		(at 53.34 210.82)
+	)
+	(no_connect
 		(at 34.29 57.15)
+	)
+	(no_connect
+		(at 53.34 204.47)
 	)
 	(no_connect
@@
 	)
 	(no_connect
+		(at 41.91 210.82)
+	)
+	(no_connect
+		(at 364.49 162.56)
+	)
+	(no_connect
 		(at 213.36 157.48)
 	)
 	(no_connect
 		(at 95.25 195.58)
+	)
+	(no_connect
+		(at 5.08 36.83)
+	)
+	(no_connect
+		(at 374.65 168.91)
+	)
+	(no_connect
+		(at 354.33 168.91)
+	)
+	(no_connect
+		(at 41.91 204.47)
 	)
 	(no_connect
@@
 	)
 	(no_connect
+		(at 5.08 24.13)
+	)
+	(no_connect
+		(at 8.89 121.92)
+	)
+	(no_connect
 		(at 46.99 57.15)
 	)
@@
 	)
 	(no_connect
+		(at 364.49 168.91)
+	)
+	(no_connect
